File: hf_pa.kicad_sch (KiCad schematic)
At the start: 66 parts, among them J12 TX_RF, J13 RX_RF, J14 TO FILT_IN, J15 TO 50Ω/50W DUMMY, J16 TO T/R, J17 TX_RF, K29 EC2-5SNU, Q10 2N2222A, Q11 2N2222A, Q12 2N2222A, Q13 2N2222A, Q14 IRF510, Q15 IRF510, Q16 2N3904, Q8 2N2222A, Q9 2N2222A, T2 Xformer, T3 Xformer, T4 Xformer

Commit message: Replaced 74hc596 parts with mcp23017 and mcp23008 parts to simplify routing and reduce external parts count.
Added interface connectors for eventualy VHF (6m/2m/1.25m) RF path board.

Attempted to create some sort of documentations...
Parts:
- renumbered C57 to C60, C58 to C61, C59 to C62, C60 to C63, C61 to C64, C62 to C65, C63 to C66, C64 to C67, C65 to C68, C66 to C69, C67 to C70, C68 to C71, C69 to C72, C70 to C73, C71 to C74, C72 to C75, D34 to D35, D35 to D36, K29 to K30, L28 to L30, L29 to L31, Q16 to Q10, Q8 to Q2, Q9 to Q3, Q10 to Q4, Q11 to Q5, Q12 to Q6, Q13 to Q7, Q14 to Q8, Q15 to Q9, R36 to R37, R37 to R38, R38 to R39, R39 to R40, R40 to R41, R41 to R42, R42 to R43, R43 to R44, R44 to R45, R45 to R46, R46 to R47, R47 to R48, R48 to R49, R49 to R50, R50 to R51, R51 to R52, R52 to R53, R53 to R54, R54 to R55, R55 to R56
Other:
- note added: "Should we abandon the ubitx PA in favor of something 100W? With bias management by uc, we can maintain 45W across HF."

Commit message: cleanup of schematic and some initial firmware works...
Parts:
- removed C60, C61, C62, C63, C64, C65, C66, C67, C68, C69, C71, C73, C74, C75: 0.1u, Capacitor_THT:C_Disc_D4.7mm_W2.5mm_P5.00mm, symbol Device:C_Small
- removed C70, C72: 470u, Capacitor_THT:CP_Radial_D4.0mm_P2.00mm, symbol Device:C_Polarized_Small_US
- removed J12: TX_RF, symbol Connector:Conn_Coaxial
- removed J15: TO 50Ω/50W DUMMY, symbol Connector:Conn_Coaxial
- removed J16: TO T/R, symbol Connector:Conn_Coaxial
- removed L30, L31: 60u, symbol Device:L
- removed Q10: 2N3904, Package_TO_SOT_THT:TO-92_Inline, symbol Transistor_BJT:2N3904
- removed Q2, Q3, Q4, Q5, Q6, Q7: 2N2222A, TO127P584H533-3, symbol 2N2222A:2N2222A
- removed Q8, Q9: IRF510, TO220, symbol IRF510:IRF510
- removed R37, R38, R46, R47: 1K, Resistor_THT:R_Axial_DIN0207_L6.3mm_D2.5mm_P2.54mm_Vertical, symbol Device:R_Small_US
- removed R39, R40, R42, R43, R44, R45, R48, R49: 22, Resistor_THT:R_Axial_DIN0207_L6.3mm_D2.5mm_P2.54mm_Vertical, symbol Device:R_Small_US
- removed R41, R50: 2.2K, Resistor_THT:R_Axial_DIN0207_L6.3mm_D2.5mm_P2.54mm_Vertical, symbol Device:R_Small_US
- removed R51, R52: 220, Resistor_THT:R_Axial_DIN0207_L6.3mm_D2.5mm_P2.54mm_Vertical, symbol Device:R_Small_US
- removed R53, R54: 47, Resistor_THT:R_Axial_DIN0207_L6.3mm_D2.5mm_P2.54mm_Vertical, symbol Device:R_Small_US
- removed R55: 1k, Resistor_THT:R_Axial_DIN0207_L6.3mm_D2.5mm_P2.54mm_Vertical, symbol Device:R_Small_US
- removed RV4, RV5: 10K, Potentiometer_THT:Potentiometer_Vishay_T7-YA_Single_Vertical, symbol Device:R_Potentiometer_Trim_US
- removed T2, T3, T4: Xformer, symbol Device:Transformer_1P_2S
- removed TP4, TP5: TX EN, symbol Connector:TestPoint
- removed TP6: PA PWR, symbol Connector:TestPoint
- removed TP7: TX_RX, symbol Connector:TestPoint_Alt
- added J19: To CTRL:ATU, symbol Connector_Generic:Conn_2Rows-09Pins
- J14: renamed from J13; value RX_RF -> TO RX_FILT_IN
- J15: renamed from J14; value TO FILT_IN -> TO ANTENNA
- J17: value TX_RF -> TO SWR_OUT
- renumbered D35 to D40, D36 to D41, K30 to K31, R56 to R47, TP8 to TP4
Connections:
- net +5V: now also J19.8 (Pin_8)
- net Earth: now also J19.6 (Pin_6)
- new net +12V: J19.4 (Pin_4)
- no-connect marks 2 -> 7
Other:
- note added: "1: 2: 3: 4: +12V 5: i2c SDA 6: GND 7: i2c SCK 8: +5V 9:"
- note removed: "Bias Adjustments"
- note removed: "Should we abandon the ubitx PA in favor of something 100W? With bias management by uc, we can maintain 45W across HF."
- moved on the sheet: D40, D41, J14, J15, J17, K31, R47, TP4
