File: radiopcb.kicad_sch (KiCad schematic)
At the start: 415 parts, among them J1 TO FILTERS IN, J10 ANTENNA, J11 TO FILTERS IN, J2 FROM PA, J3 TO FILTERS OUT, J4 RX_RF, J5 To CTRL:FILT, J6 USB, J7 FILTERS OUT, J8 FILTERS IN, J9 USB_A_Stacked, K1 EC2-5SNU, K2 EC2-5SNU, K3 EC2-5SNU, K4 EC2-5SNU, K5 EC2-5SNU, K6 EC2-5SNU, K7 EC2-5SNU, K8 EC2-5SNU, K9 EC2-5SNU, Q1 2N2222A, Q10 IRF510, Q11 IRF510, Q12 2N3904, Q2 2N2222A, Q3 BT169B, Q5 2N2222A, Q6 2N2222A, Q7 2N2222A, Q8 2N2222A, T1 Xformer, T2 Xformer, T3 Xformer, U1 ULN2804A, U10 LM1117-ADJ, U11 TPS563201DDCR, U12 LM1117-ADJ, U13 BlackPill_STLINK, U2 74HC596, U3 LM555xM, U4 74HC596, U5 ULN2804A, U6 74HC596, U7 ULN2804A, U8 TUSB4041I, U9 CM119B, Y1 24Mhz

Commit message: cleanup
Parts:
- removed C32, C33, C35, C37, C38, C65, C66, C67, C? (x21): 100n, symbol Device:C_Small
- removed C64, C68: 0.1u, Capacitor_THT:C_Disc_D4.7mm_W2.5mm_P5.00mm, symbol Device:C_Small
- removed D15, D16, D17, D18, D20, D32, D33, D34, D6, D? (x20): 1N4007, Diode_THT:D_DO-41_SOD81_P10.16mm_Horizontal, symbol Diode:1N4007
- removed D24, D25, D26, D27, D28, D29, D30, D31, D35, D37, D4, D? (x19): 1N4001, Diode_THT:D_DO-41_SOD81_P10.16mm_Horizontal, symbol Diode:1N4001
- removed D5: 160M-Green, symbol Device:LED
- removed D?: HiZ-Green, symbol Device:LED
- removed D?: AT-10pf, symbol Device:LED
- removed K9: EC2-5SNU, Relay_THT:Relay_DPDT_Kemet_EC2, symbol Relay:EC2-5SNU
- removed K?: G6E, Relay_THT:Relay_SPDT_Omron_G6E, symbol Relay:G6E
- removed R24, R?: 1K, symbol Device:R_Small_US
- removed R?: 10k, symbol Device:R_Small_US
- removed RL1, RL?: T/R, Relay_THT:Relay_DPDT_Panasonic_JW2, symbol Relay:JW2
- removed U1, U5, U7, U?: ULN2804A, Package_DIP:DIP-18_W7.62mm_LongPads, symbol Transistor_Array:ULN2804A
- added C61: 120p, symbol Device:C_Small
- added C74: 36p, symbol Device:C_Small
- added C77, C79, C80: 0.1u, Capacitor_THT:C_Disc_D4.7mm_W2.5mm_P5.00mm, symbol Device:C_Small
- added C?: 100u, symbol Device:C_Polarized_US
- added D38: 6M-Green, symbol Device:LED
- added D70: HiZ-Green, symbol Device:LED
- added D?: 1N4001, Diode_THT:D_DO-41_SOD81_P10.16mm_Horizontal, symbol Diode:1N4001
- added J12: To CTRL:FILT_H, symbol Connector_Generic:Conn_2Rows-09Pins
- added J18: CTRL:ATU_H, symbol Connector_Generic:Conn_2Rows-09Pins
- added J19: CTRL:FILT_H, symbol Connector_Generic:Conn_2Rows-09Pins
- added J? (x2): UF1_OUT, symbol Connector:Conn_Coaxial
- added K10: EC2-5SNU, Relay_THT:Relay_DPDT_Kemet_EC2, symbol Relay:EC2-5SNU
- added K28, K?: G6E, Relay_THT:Relay_SPDT_Omron_G6E, symbol Relay:G6E
- added L18, L22: 240n, symbol Device:L_Ferrite
- added Q13, Q14: 2N3904, Package_TO_SOT_THT:TO-92_Inline, symbol Transistor_BJT:2N3904
- added R39, R52: 10k, symbol Device:R_Small_US
- added U14: ULN2804A, Package_DIP:DIP-18_W7.62mm_LongPads, symbol Transistor_Array:ULN2804A
- added U15: 74HC596, Package_SO:TSSOP-16_4.4x5mm_P0.65mm, symbol 74xx:74HC596
- added U? (x4): ULN2803A, symbol Transistor_Array:ULN2803A
- C31: value 100n -> 36p
- D13: value 6M-Green -> USER-Green
- D79: renamed from D?; value AT-880pF -> AT-1.25uH
- D80: renamed from D?; value AT-440pF -> AT-2.5uH
- D81: renamed from D?; value AT-220pF -> AT-5.0uH
- D82: renamed from D?; value AT-220pF -> AT-10uH
- D92: renamed from D?; value AT-440pF -> AT-0.22uH
- D93: renamed from D?; value AT-220pF -> AT-0.39uH
- D94: renamed from D?; value AT-100pf -> AT-0.59uH
- D97: renamed from D?; value AT-10pf -> BAND_SPLIT
- J1: value TO FILTERS IN -> TO T/R
- J10: value ANTENNA -> TO SWR_IN
- J11: value TO FILTERS IN -> TO FILT_OUT
- J13: renamed from J?; value IN -> SWR_IN
- J14: renamed from J?; value OUT -> TO ANTENNA
- J16: renamed from J?; value CTRL:FILT -> CTRL:ATU_L
- J17: renamed from J?; value CTRL:ATU -> CTRL:FILT_L
- J3: value TO FILTERS OUT -> TO FILT_IN
- J5: value To CTRL:FILT -> To CTRL:FILT_L
- J7: value FILTERS OUT -> FILT_OUT
- J8: value FILTERS IN -> FILT_IN
- L23: renamed from L?; value 3.3u -> 1.25u
- L24: renamed from L?; value 3.3u -> 2.5u
- L25: renamed from L?; value 3.3u -> 5.0u
- L26: renamed from L?; value 3.3u -> 10u
- L27: renamed from L?; value 3.3u -> 0.11u
- L28: renamed from L?; value 3.3u -> 0.22u
- L29: renamed from L?; value 3.3u -> 0.39u
- L30: renamed from L?; value 3.3u -> 0.59u
- gave numbers to parts that had none: 94
Connections:
- net +12V: now also C63.2, C70.2, C72.2, C82.2, D36.2 (A), D50.2 (A), D51.2 (A), D52.2 (A), D53.2 (A), D64.2 (A), D65.2 (A), D66.2 (A), D67.2 (A), D79.2 (A), D80.2 (A), D81.2 (A), D82.2 (A), D91.2 (A), D92.2 (A), D93.2 (A), D94.2 (A), K1.1, K11.1, K12.1, K13.1, K14.1, K15.1, K16.1, K17.1, K18.1, K19.1, K2.1, K20.1, K21.1, K22.1, K23.1, K24.1, K25.1, K26.1, K3.1, K4.1, K5.1, K6.1, K7.1, K8.1, R25.1, R26.1, R27.1, R31.1, R34.1, R35.1, R36.1, R37.1, RL2.8, D70.2 (A), K?.1, U?.10 (COM), U?.10 (COM), U?.10 (COM)
- net +5V: now also K9.1, R24.1, U2.16 (VCC), J18.8 (Pin_8), J19.8 (Pin_8), K10.1, R39.1; no longer C70.2, C82.2
- net Earth: now also R21.1, C77.1, C79.1, C80.1, D?.2 (A), J12.6 (Pin_6), J18.6 (Pin_6), J19.6 (Pin_6), K28.6, U14.9 (GND), U15.8 (GND), U?.9 (GND), U?.9 (GND), U?.9 (GND), U?.9 (GND); no longer D2.1 (K), J5.6 (Pin_6)
- net GND: now also C104.2, C105.2, C71.1, C72.1, C61.2, C74.2, C?.2, J?.2 (Ext), J?.2 (Ext); no longer C104.1, D10.1 (K), D11.1 (K), D12.1 (K), D13.1 (K), D14.1 (K), D50.1 (K), D51.1 (K), D52.1 (K), D53.1 (K), D6.1 (K), D64.1 (K), D65.1 (K), D66.1 (K), D67.1 (K), D7.1 (K), D79.1 (K), D8.1 (K), D80.1 (K), D81.1 (K), D82.1 (K), D9.1 (K), D91.1 (K), D92.1 (K), D93.1 (K), D94.1 (K), K1.12, K11.1, K12.1, K13.1, K14.1, K15.1, K16.1, K17.1, K18.1, K19.1, K2.12, K20.1, K21.1, K22.1, K23.1, K24.1, K25.1, K26.1, K3.12, K4.12, K5.12, K6.12, K7.12, K8.12, K9.12
- net at C71.2, J15.8 (Pin_8), U6.16 (VCC): now also C?.1; no longer C72.2
- net at TP16.1: now also D2.2 (A), D?.1 (K), K28.1; no longer R21.1
- net at K19.10: now also L23.2, RL2.5, K?.12
- net at K19.6, R53.1: now also U?.14 (O5)
- net at K19.7: now also K20.10, L23.1, L24.2
- net at K16.6, R46.1: now also U?.17 (O2)
- net at R45.2: now also D64.1 (K); no longer D64.2 (A)
- net at R59.2: now also D81.1 (K); no longer D81.2 (A)
- net at R38.1, RL2.1: now also U?.17 (O2)
- net at D36.1 (K): now also R38.2; no longer RL2.8
- net at K17.6, R47.1: now also U?.16 (O3)
- net at R62.2: now also D92.1 (K); no longer D92.2 (A)
- net at R47.2: now also D66.1 (K); no longer D66.2 (A)
- net at R54.2: now also D80.1 (K); no longer D80.2 (A)
- net at L27.1: now also K23.10; no longer L23.2
- net at L24.1, L25.1: now also K20.7, K21.10
- net at R61.2: now also D91.1 (K); no longer D91.2 (A)
- net at R43.2: now also D53.1 (K); no longer D53.2 (A)
- net at U4.1 (QB): now also U?.2 (I2)
- net at U4.15 (QA): now also U?.1 (I1)
- net at U4.2 (QC): now also U?.3 (I3)
- net at U4.3 (QD): now also U?.4 (I4)
- net at U4.4 (QE): now also U?.5 (I5)
- net at U4.5 (QF): now also U?.6 (I6)
- net at U4.6 (QG): now also U?.7 (I7)
- net at U4.7 (QH): now also U?.8 (I8)
- net at K25.6, R63.1: now also U?.16 (O3)
- net at R63.2: now also D93.1 (K); no longer D93.2 (A)
- net at K12.6, R41.1: now also U?.13 (O6)
- net at K20.6, R54.1: now also U?.13 (O6)
- net at U16.1 (QB): now also U?.2 (I2)
- net at U16.15 (QA): now also U?.1 (I1)
- net at U16.2 (QC): now also U?.3 (I3)
- net at U16.3 (QD): now also U?.4 (I4)
- net at U16.4 (QE): now also U?.5 (I5)
- net at U16.5 (QF): now also U?.6 (I6)
- net at U16.6 (QG): now also U?.7 (I7)
- net at U16.7 (QH): now also U?.8 (I8)
- net at K11.6, R40.1: now also U?.14 (O5)
- net at R41.2: now also D51.1 (K); no longer D51.2 (A)
- net at K14.6, R43.1: now also U?.11 (O8)
- net at K11.7, K12.7, K13.7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: now also K?.7; no longer RL2.5
- net at K26.6, R64.1: now also U?.15 (O4)
- net at K22.10: now also K21.7, L25.2, L26.1
- net at K22.6, R60.1: now also U?.11 (O8)
- net at K22.7: now also K26.7, L26.2, L30.2, RL2.4, K?.10
- net at K23.6, R61.1: now also U?.18 (O1)
- net at U2.1 (QB): now also U?.7 (I7)
- net at U2.15 (QA): now also U?.8 (I8)
- net at U2.2 (QC): now also U?.6 (I6)
- net at U2.3 (QD): now also U?.5 (I5)
- net at U2.4 (QE): now also U?.4 (I4)
- net at U2.5 (QF): now also U?.3 (I3)
- net at U2.6 (QG): now also U?.2 (I2)
- net at U2.7 (QH): now also U?.1 (I1)
- net at K25.10: now also K24.7, L28.2, L29.1
- net at K25.7: now also K26.10, L29.2, L30.1
- net at R46.2: now also D65.1 (K); no longer D65.2 (A)
- net at K21.6, R59.1: now also U?.12 (O7)
- net at C105.1, K15.12: now also C104.1
- net at K23.7: now also K24.10, L27.2, L28.1
- net at K24.6, R62.1: now also U?.17 (O2)
- net at R60.2: now also D82.1 (K); no longer D82.2 (A)
- net at R40.2: now also D50.1 (K); no longer D50.2 (A)
- net at K13.6, R42.1: now also U?.12 (O7)
- net at R42.2: now also D52.1 (K); no longer D52.2 (A)
- net at K15.6, R45.1: now also U?.18 (O1)
- net at J4.1 (In): now also K28.10
- net at J2.1 (In): now also K28.12
- net at K8.5: now also J?.1 (In)
- net at K8.8: now also J?.1 (In)
- net at R21.2: now also D2.1 (K); no longer D2.2 (A)
- net at R64.2: now also D94.1 (K); no longer D94.2 (A)
- net at K18.6, R48.1: now also U?.15 (O4)
- net at R48.2: now also D67.1 (K); no longer D67.2 (A)
- net at C31.1: now also K10.5, L18.2
- net at R53.2: now also D79.1 (K); no longer D79.2 (A)
- net at J3.1 (In): now also K28.7
- net at U6.1 (QB): now also U?.2 (I2)
- net at U6.15 (QA): now also U?.1 (I1)
- net at U6.2 (QC): now also U?.3 (I3)
- net at U6.3 (QD): now also U?.4 (I4)
- net at U6.4 (QE): now also U?.5 (I5)
- net at U6.5 (QF): now also U?.6 (I6)
- net at U6.6 (QG): now also U?.7 (I7)
- net at U6.7 (QH): now also U?.8 (I8)
- new net: C74.1, K10.8, L22.1
- new net: U14.1 (I1), U15.15 (QA)
- new net: C77.2, C79.2, C80.2, J12.8 (Pin_8), U14.10 (COM), U15.16 (VCC)
- new net: D6.1 (K), K9.12, U14.11 (O8)
- new net: D38.1 (K), K10.12, U14.12 (O7)
- new net: U14.2 (I2), U15.1 (QB)
- new net: U14.3 (I3), U15.2 (QC)
- new net: U14.4 (I4), U15.3 (QD)
- new net: U14.5 (I5), U15.4 (QE)
- new net: U14.6 (I6), U15.5 (QF)
- new net: U14.7 (I7), U15.6 (QG)
- new net: U14.8 (I8), U15.7 (QH)
- new net: D14.1 (K), K1.12, U?.11 (O8)
- new net: D13.1 (K), K8.12, U?.12 (O7)
- new net: D12.1 (K), K7.12, U?.13 (O6)
- new net: D11.1 (K), K6.12, U?.14 (O5)
- new net: D10.1 (K), K5.12, U?.15 (O4)
- new net: D9.1 (K), K4.12, U?.16 (O3)
- new net: D8.1 (K), K3.12, U?.17 (O2)
- new net: D7.1 (K), K2.12, U?.18 (O1)
- new net: J18.5 (Pin_5), J19.5 (Pin_5)
- new net: J18.7 (Pin_7), J19.7 (Pin_7)
- new net: C61.1, L18.1, L22.2
- new net: K?.6, R52.1, U?.18 (O1)
- new net: J12.1 (Pin_1), U15.13 (~{OE})
- new net: J12.5 (Pin_5), U15.10 (~{SRCLR})
- new net: J12.7 (Pin_7), U15.11 (SRCLK), U15.12 (RCLK)
- new net: J12.9 (Pin_9), U15.14 (SER)
- new net: D38.2 (A), R39.2
- new net: K10.10, K10.3
- new net: D70.1 (K), R52.2
- now unconnected: J15.6 (Pin_6), J5.8 (Pin_8)
Other:
- note added: "***TODO*** Add solder jumpers to bypass HUB if not built"
- note added: "2M <152Mhz"
- note added: "6M <60Mhz"
- note added: "HIGH"
- note added: "High Band"
- note added: "LOW"
- note added: "LOW/HI BAND"
- note added: "MW HPF >1.7Mhz"
- note added: "Optional User filter"
- note added: "TODO: * Verify component values - LED resistors - 1.1/3.3V psu ext."
- note removed: "6M <54Mhz"
- note removed: "GRAVEYARD"
- note removed: "HF"
- note removed: "HF/VHF"
- note removed: "MW HPF >1.8Mhz"
- note removed: "TODO: * Fix relay coil 'polarities' * Verify component values * Move 6M filter to VHF section"
- note removed: "VHF"
- moved on the sheet: C11, C12, C14, C16, C17, C20, C24, C3, C34, C5, C51, C52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

Commit message: cleanup
Parts:
- removed C1, C2: 10u, Capacitor_THT:CP_Radial_D4.0mm_P2.00mm, symbol Device:C_Polarized_Small_US
- removed C10, C15, C18, C19, C21, C22, C23, C26, C28, C29, C30, C36, C4, C44, C45, C54, C62, C63, C69, C70, C71, C72, C8, C81, C82, C9: 0.1u, Capacitor_THT:C_Disc_D4.7mm_W2.5mm_P5.00mm, symbol Device:C_Small
- removed C101, C103, C95, C96: 0.01, symbol Device:C_Small
- removed C102: 3-23, symbol Device:C_Variable
- removed C104, C105, C106, C107, C108, C89: 10p, symbol Device:C_Small
- removed C109: 39p, symbol Device:C_Small
- removed C11, C59: 110p, symbol Device:C_Small
- removed C110: 100, symbol Device:C_Small
- removed C12, C60: 68p, symbol Device:C_Small
- removed C120: 100n, symbol Device:C_Small
- removed C14, C34: 1.3n, symbol Device:C_Small
- removed C16: 3.3n, symbol Device:C_Small
- removed C17: 1.6n, symbol Device:C_Small
- removed C20: 910p, symbol Device:C_Small
- removed C24: 620p, symbol Device:C_Small
- removed C25, C27: 470u, Capacitor_THT:CP_Radial_D4.0mm_P2.00mm, symbol Device:C_Polarized_Small_US
- removed C3, C55: 1.0n, symbol Device:C_Small
- removed C39, C40, C41, C42, C43: 10u, Capacitor_THT:C_Disc_D4.7mm_W2.5mm_P5.00mm, symbol Device:C_Small
- removed C46, C47: 100n, Capacitor_THT:C_Disc_D4.7mm_W2.5mm_P5.00mm, symbol Device:C_Small
- removed C48: 47u, Capacitor_THT:C_Disc_D4.7mm_W2.5mm_P5.00mm, symbol Device:C_Small
- removed C49, C50: 220u, Capacitor_THT:CP_Radial_D4.0mm_P2.00mm, symbol Device:C_Polarized_Small_US
- removed C5, C56: 510p, symbol Device:C_Small
- removed C51: 360p, symbol Device:C_Small
- removed C52, C90: 220p, symbol Device:C_Small
- removed C57, C6: 270p, symbol Device:C_Small
- removed C58, C7: 200p, symbol Device:C_Small
- removed C87, C93: 82p, symbol Device:C_Small
- removed C88: 150p, symbol Device:C_Small
- removed C91: 100p, symbol Device:C_Small
- removed C92: 560p, symbol Device:C_Small
- removed C?: 100u, symbol Device:C_Polarized_US
- removed D1, D21, D22, D23, D?: 1N4001, Diode_THT:D_DO-41_SOD81_P10.16mm_Horizontal, symbol Diode:1N4001
- removed D10: 30M-Green, symbol Device:LED
- removed D11: 17M-Green, symbol Device:LED
- removed D12: 10M-Green, symbol Device:LED
- removed D13: USER-Green, symbol Device:LED
- removed D14: MW HPF-Green, symbol Device:LED
- removed D19: LED-Green, LED_SMD:LED_PLCC_2835_Handsoldering, symbol Device:LED
- removed D2: TX-Red, symbol Device:LED
- removed D3: LED, symbol Device:LED
- removed D36: Bypass-Red, symbol Device:LED
- removed D50: AT-82pF, symbol Device:LED
- removed D51: AT-160pF, symbol Device:LED
- removed D52: AT-320pF, symbol Device:LED
- removed D53: AT-642pF, symbol Device:LED
- removed D58, D63: 1N4148, Diode_THT:D_DO-35_SOD27_P7.62mm_Horizontal, symbol Diode:1N4148
- removed D64: AT-5pF, symbol Device:LED
- removed D65: AT-10pF, symbol Device:LED
- removed D66: AT-20pF, symbol Device:LED
- removed D67: AT-39pF, symbol Device:LED
- removed D7: 160M-Green, symbol Device:LED
- removed D70: HiZ-Green, symbol Device:LED
- removed D79: AT-1.25uH, symbol Device:LED
- removed D8: 80M-Green, symbol Device:LED
- removed D80: AT-2.5uH, symbol Device:LED
- removed D81: AT-5.0uH, symbol Device:LED
- removed D82: AT-10uH, symbol Device:LED
- removed D9: 40M-Green, symbol Device:LED
- removed D91: AT-0.11uH, symbol Device:LED
- removed D92: AT-0.22uH, symbol Device:LED
- removed D93: AT-0.39uH, symbol Device:LED
- removed D94: AT-0.59uH, symbol Device:LED
- removed D95: 1N4007, Diode_THT:D_DO-41_SOD81_P10.16mm_Horizontal, symbol Diode:1N4007
- removed F1, F2: 30A, Fuse:Fuseholder_Blade_Mini_Keystone_3568, symbol Device:Fuse_Small
- removed F3, F4: 5A, Fuse:Fuseholder_Blade_Mini_Keystone_3568, symbol Device:Fuse_Small
- removed F5, F8: 3A, Fuse:Fuseholder_Blade_Mini_Keystone_3568, symbol Device:Fuse_Small
- removed F6, F7: 250mA, Fuse:Fuseholder_Blade_Mini_Keystone_3568, symbol Device:Fuse_Small
- removed J1: TO T/R, symbol Connector:Conn_Coaxial
- removed J10: TO SWR_IN, symbol Connector:Conn_Coaxial
- removed J11: TO FILT_OUT, symbol Connector:Conn_Coaxial
- removed J13: SWR_IN, symbol Connector:Conn_Coaxial
- removed J14: TO ANTENNA, symbol Connector:Conn_Coaxial
- removed J15: To CTRL:ATU, symbol Connector_Generic:Conn_2Rows-09Pins
- removed J16: CTRL:ATU_L, symbol Connector_Generic:Conn_2Rows-09Pins
- removed J17: CTRL:FILT_L, symbol Connector_Generic:Conn_2Rows-09Pins
- removed J18: CTRL:ATU_H, symbol Connector_Generic:Conn_2Rows-09Pins
- removed J19: CTRL:FILT_H, symbol Connector_Generic:Conn_2Rows-09Pins
- removed J2: FROM PA, symbol Connector:Conn_Coaxial
- removed J3: TO FILT_IN, symbol Connector:Conn_Coaxial
- removed J4: RX_RF, symbol Connector:Conn_Coaxial
- removed J5: To CTRL:FILT_L, symbol Connector_Generic:Conn_2Rows-09Pins
- removed J6: USB, Connector_USB:USB_C_Receptacle_Molex_105450-0101, symbol Connector:USB_C_Receptacle_USB2.0
- removed J7: FILT_OUT, symbol Connector:Conn_Coaxial
- removed J8: FILT_IN, symbol Connector:Conn_Coaxial
- removed J9: USB_A_Stacked, symbol Connector:USB_A_Stacked
- removed J? (x2): UF1_OUT, symbol Connector:Conn_Coaxial
- removed K1, K2, K3, K4, K5, K6, K7, K8: EC2-5SNU, Relay_THT:Relay_DPDT_Kemet_EC2, symbol Relay:EC2-5SNU
- removed K11, K12, K13, K14, K15, K16, K17, K18, K19, K20, K21, K22, K23, K24, K25, K26, K28, K?: G6E, Relay_THT:Relay_SPDT_Omron_G6E, symbol Relay:G6E
- removed L1, L2: 60u, symbol Device:L
- removed L11: 2.2u, symbol Device:L_Ferrite
- removed L12, L4: 6.2u, symbol Device:L_Ferrite
- removed L13, L5: 3.3u, symbol Device:L_Ferrite
- removed L14, L6: 1.8u, symbol Device:L_Ferrite
- removed L15: 1.3, symbol Device:L_Ferrite
- removed L16, L8: 680n, symbol Device:L_Ferrite
- removed L17, L9: 430n, symbol Device:L_Ferrite
- removed L19, L20: 3.9u, symbol Device:L_Ferrite
- removed L23: 1.25u, symbol Device:L_Ferrite
- removed L24: 2.5u, symbol Device:L_Ferrite
- removed L25: 5.0u, symbol Device:L_Ferrite
- removed L26: 10u, symbol Device:L_Ferrite
- removed L27: 0.11u, symbol Device:L_Ferrite
- removed L28: 0.22u, symbol Device:L_Ferrite
- removed L29: 0.39u, symbol Device:L_Ferrite
- removed L3: 3.3uH, symbol Device:L
- removed L30: 0.59u, symbol Device:L_Ferrite
- removed L7: 1.3u, symbol Device:L_Ferrite
- removed Q1, Q2, Q5, Q6, Q7, Q8: 2N2222A, TO127P584H533-3, symbol 2N2222A:2N2222A
- removed Q10, Q11: IRF510, TO220, symbol IRF510:IRF510
- removed Q12, Q15, Q16, Q4, Q9: 2N3904, Package_TO_SOT_THT:TO-92_Inline, symbol Transistor_BJT:2N3904
- removed Q3: BT169B, Package_TO_SOT_THT:TO-92_Inline, symbol Triac_Thyristor:BT169B
- removed R10, R23: R_Small_US, symbol Device:R_Small_US
- removed R11, R12, R15, R16, R19, R20, R5, R6: 22, Resistor_THT:R_Axial_DIN0207_L6.3mm_D2.5mm_P2.54mm_Vertical, symbol Device:R_Small_US
- removed R13, R14: 10, symbol Device:R_Small_US
- removed R17, R18, R3, R4: 1K, Resistor_THT:R_Axial_DIN0207_L6.3mm_D2.5mm_P2.54mm_Vertical, symbol Device:R_Small_US
- removed R21, R25, R26, R27, R31, R34, R35, R36, R37, R38, R52: 10k, symbol Device:R_Small_US
- removed R22, R9: 2.2K, Resistor_THT:R_Axial_DIN0207_L6.3mm_D2.5mm_P2.54mm_Vertical, symbol Device:R_Small_US
- removed R28, R29: 220, Resistor_THT:R_Axial_DIN0207_L6.3mm_D2.5mm_P2.54mm_Vertical, symbol Device:R_Small_US
- removed R30, R32: 47, Resistor_THT:R_Axial_DIN0207_L6.3mm_D2.5mm_P2.54mm_Vertical, symbol Device:R_Small_US
- removed R33: 1k, Resistor_THT:R_Axial_DIN0207_L6.3mm_D2.5mm_P2.54mm_Vertical, symbol Device:R_Small_US
- removed R40, R41, R42, R43, R45, R46, R47, R48, R53, R54, R59, R60, R61, R62, R63, R64: 1K, symbol Device:R_Small_US
- removed R44, R50: 100, symbol Device:R_Small_US
- removed R49: 150, symbol Device:R_Small_US
- removed R51: 3.3k, symbol Device:R_Small_US
- removed R55: 9.53K, Resistor_THT:R_Axial_DIN0207_L6.3mm_D2.5mm_P2.54mm_Vertical, symbol Device:R_Small_US
- removed R56, R7, R8: 10M, Resistor_THT:R_Axial_DIN0207_L6.3mm_D2.5mm_P2.54mm_Vertical, symbol Device:R_Small_US
- removed R57: 10k, Resistor_THT:R_Axial_DIN0207_L6.3mm_D2.5mm_P2.54mm_Vertical, symbol Device:R_Small_US
- removed R58: 54.9k, Resistor_THT:R_Axial_DIN0207_L6.3mm_D2.5mm_P2.54mm_Vertical, symbol Device:R_Small_US
- removed RL2: T/R, Relay_THT:Relay_DPDT_Panasonic_JW2, symbol Relay:JW2
- removed RV1, RV2: 10K, Potentiometer_THT:Potentiometer_Vishay_T7-YA_Single_Vertical, symbol Device:R_Potentiometer_Trim_US
- removed RV3: R_Potentiometer_US, symbol Device:R_Potentiometer_US
- removed RV4, RV5: 100k, symbol Device:R_Potentiometer_US
- removed T1, T2, T3: Xformer, symbol Device:Transformer_1P_2S
- removed T4: Transformer_1P_SS, symbol Device:Transformer_1P_SS
- removed TP1: TX_RF, symbol Connector:TestPoint
- removed TP11, TP7: TX EN, symbol Connector:TestPoint
- removed TP14: PA PWR, symbol Connector:TestPoint
- removed TP15, TP16: TX_RX, symbol Connector:TestPoint_Alt
- removed TP17: TX_AF, symbol Connector:TestPoint_Alt
- removed TP18: RX_AF_I, symbol Connector:TestPoint_Alt
- removed TP2: WDT Out, symbol Connector:TestPoint_Alt
- removed TP3: FWD, symbol Connector:TestPoint
- removed TP4: REV, symbol Connector:TestPoint
- removed TP5: RX_AF_Q, symbol Connector:TestPoint_Alt
- removed U10, U12: LM1117-ADJ, symbol Regulator_Linear:LM1117-ADJ
- removed U11: TPS563201DDCR, SOT95P280X110-6N, symbol TPS563201DDCR:TPS563201DDCR
- removed U13: BlackPill_STLINK, blackpill:BlackPill_STLINK, symbol blackpill_stlink:BlackPill_STLINK
- removed U16, U2, U4, U6: 74HC596, Package_SO:TSSOP-16_4.4x5mm_P0.65mm, symbol 74xx:74HC596
- removed U3: LM555xM, Package_SO:SOIC-8_3.9x4.9mm_P1.27mm, symbol Timer:LM555xM
- removed U8: TUSB4041I, Package_QFP:HTQFP-64-1EP_10x10mm_P0.5mm_EP8x8mm_Mask4.4x4.4mm_ThermalVias, symbol Interface_USB:TUSB4041I
- removed U9: CM119B, Package_QFP:TQFP-48_7x7mm_P0.5mm, symbol CM119B:CM119B
- removed U? (x4): ULN2803A, symbol Transistor_Array:ULN2803A
- removed Y1: 24Mhz, Crystal:Crystal_SMD_HC49-SD_HandSoldering, symbol Device:Crystal_GND2_Small
- added D1: LED, symbol Device:LED
- added Q1: BT169B, Package_TO_SOT_THT:TO-92_Inline, symbol Triac_Thyristor:BT169B
- added RV1: R_Potentiometer_US, symbol Device:R_Potentiometer_US
- added TP1: WDT Out, symbol Connector:TestPoint_Alt
- added U1: LM555xM, Package_SO:SOIC-8_3.9x4.9mm_P1.27mm, symbol Timer:LM555xM
- R1, R2: value 10M -> R_Small_US; footprint Resistor_THT:R_Axial_DIN0207_L6.3mm_D2.5mm_P2.54mm_Vertical -> (none)
- renumbered C13 to C1, C31 to C2, C53 to C3, C61 to C4, C73 to C5, C74 to C6, C77 to C7, C79 to C8, C80 to C9, D6 to D2, D38 to D3, D96 to D4, D97 to D5, J12 to J1, K9 to K1, K10 to K2, K27 to K3, L10 to L1, L18 to L2, L21 to L3, L22 to L4, Q13 to Q2, Q14 to Q3, R24 to R3, R39 to R4, R65 to R5, U14 to U2, U15 to U3
Connections:
- net GND: now also D1.1 (K), U1.1 (GND); no longer R2.2
- net at R1.2: no longer R2.1
- net at R1.1: now also RV1.2
- new net: D1.2 (A), R2.2
- new net: Q1.3 (K), R2.1, TP1.1
- no-connect marks 18 -> 0
Other:
- added sheet Control Logic (control_logic.kicad_sch)
- added sheet HF ATU (hf_atu.kicad_sch)
- added sheet HF Filters (hf_filters.kicad_sch)
- added sheet HF PA (hf_pa.kicad_sch)
- added sheet Power Supply (psu.kicad_sch)
- note added: "I'm a KiCad noob. How do i make these autoupdate? Double click the sheets below to open."
- note added: "This section contains the Antenna Matching unit for HF at 100W"
- note added: "This section contains the LPF and HPF filters for cleaning up PA output. 100W continuous maximum"
- note added: "This section contains the control logic and USB interface"
- note added: "This section contains the our HF power amplifier. Output is up to 45W, if bias managed"
- note added: "This section contains the power supplies"
- note removed: "!!! VERIFY THESE VALUES !!!"
- note removed: "***TODO*** Add solder jumpers to bypass HUB if not built"
- note removed: "1.1V"
- note removed: "15-10M <32Mhz"
- note removed: "160M <2.5Mhz"
- note removed: "1: CS 2: NC 3: OE 4: NC 5: CLR 6: GND 7: CLK 8: +5V 9: SER_OUT"
- note removed: "20-17M <24Mhz"
- note removed: "3.3V"
- note removed: "30M <13Mhz"
- note removed: "40M <7.3Mhz"
- note removed: "80M <5.0Mhz"
- note removed: "BYPASS"
- note removed: "Bias Adjustments"
- note removed: "Bypasses the entire tuner to reduce losses."
- note removed: "Capacitive"
- note removed: "Control Interface"
- note removed: "HF Antenna Matching Unit"
- note removed: "HF LPF/HPF Filters"
- note removed: "HF Power Amplifier"
- note removed: "HF RF Section (PCB002)"
- note removed: "HF T/R Switching"
- note removed: "HI-Z"
- note removed: "Host Interface"
- note removed: "Inductive"
- note removed: "Input"
- note removed: "MW HPF >1.7Mhz"
- note removed: "Optional User filter"
- note removed: "Output"
- note removed: "PSU/Control (PCB001)"
- note removed: "Power Supply"
- note removed: "RF Frontend (PCB003)"
- note removed: "SWR BRIDGE"
- note removed: "Switches C between in/out sides of L network."
- note removed: "T30-6"
- note removed: "TRANSMIT"
- note removed: "Update all these to reflect raised cutoffs to avoid IMD"
- note removed: "VHF RF Section (PCB004)"
- title: tinytrx -> Radio Project
- moved on the sheet: C1, C2, C3, C4, C5, C6, C7, C8, C9, D2, D3, D4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

Commit message: Replaced 74hc596 parts with mcp23017 and mcp23008 parts to simplify routing and reduce external parts count.
Added interface connectors for eventualy VHF (6m/2m/1.25m) RF path board.

Attempted to create some sort of documentations...
Parts:
- removed C1, C2, C5, C6: 36p, symbol Device:C_Small
- removed C3, C4: 120p, symbol Device:C_Small
- removed C7, C8, C9: 0.1u, Capacitor_THT:C_Disc_D4.7mm_W2.5mm_P5.00mm, symbol Device:C_Small
- removed D1: LED, symbol Device:LED
- removed D2, D3: 6M-Green, symbol Device:LED
- removed D4: 1N4001, Diode_THT:D_DO-41_SOD81_P10.16mm_Horizontal, symbol Diode:1N4001
- removed D5: BAND_SPLIT, symbol Device:LED
- removed J1: To CTRL:FILT_H, symbol Connector_Generic:Conn_2Rows-09Pins
- removed K1, K2: EC2-5SNU, Relay_THT:Relay_DPDT_Kemet_EC2, symbol Relay:EC2-5SNU
- removed K3: G6E, Relay_THT:Relay_SPDT_Omron_G6E, symbol Relay:G6E
- removed L1, L2, L3, L4: 240n, symbol Device:L_Ferrite
- removed Q1: BT169B, Package_TO_SOT_THT:TO-92_Inline, symbol Triac_Thyristor:BT169B
- removed Q2, Q3: 2N3904, Package_TO_SOT_THT:TO-92_Inline, symbol Transistor_BJT:2N3904
- removed R1, R2: R_Small_US, symbol Device:R_Small_US
- removed R3, R4: 10k, symbol Device:R_Small_US
- removed R5: 1K, symbol Device:R_Small_US
- removed RV1: R_Potentiometer_US, symbol Device:R_Potentiometer_US
- removed TP1: WDT Out, symbol Connector:TestPoint_Alt
- removed U1: LM555xM, Package_SO:SOIC-8_3.9x4.9mm_P1.27mm, symbol Timer:LM555xM
- removed U2: ULN2804A, Package_DIP:DIP-18_W7.62mm_LongPads, symbol Transistor_Array:ULN2804A
- removed U3: 74HC596, Package_SO:TSSOP-16_4.4x5mm_P0.65mm, symbol 74xx:74HC596
Other:
- added sheet VHF (vhf.kicad_sch)
- note added: "This section contains the Antenna Matching unit for HF at 50W 100% duty cycle"
- note added: "This section contains the LPF and HPF filters for cleaning up PA output. 50W 100% duty cycle"
- note removed: "2M <152Mhz"
- note removed: "5V"
- note removed: "6M <60Mhz"
- note removed: "Can we do anything here to improve the serial shielding?"
- note removed: "FRONTEND"
- note removed: "Filter Control"
- note removed: "Fine Adjust"
- note removed: "HIGH"
- note removed: "High Band"
- note removed: "I'm a KiCad noob. How do i make these autoupdate? Double click the sheets below to open."
- note removed: "LOW"
- note removed: "LOW/HI BAND"
- note removed: "Socketed"
- note removed: "TODO: * Verify component values - LED resistors - 1.1/3.3V psu ext."
- note removed: "TX Watchdog"
- note removed: "This section contains the Antenna Matching unit for HF at 100W"
- note removed: "This section contains the LPF and HPF filters for cleaning up PA output. 100W continuous maximum"
- note removed: "To prevent runaway TX, require host CPU to toggle WD pin >100ms, before timeout. This should be rather lengthy, perhaps 5-10 minutes, as it will define the maximum allowed TX time in self-hosted modes. This should have a direct unmuxed GPIO pin"
- note removed: "WDT Triggered"

Commit message: cleanup of schematic and some initial firmware works...
Other:
- sheet VHF renamed VHF_Filters
- added sheet HF Legal Limit Amp (hf_amp_legal_limit.kicad_sch)
- added sheet graveyard (graveyard.kicad_sch)
