File: vhf.kicad_sch (KiCad schematic)
At the start: 41 parts

Commit message: cleanup of schematic and some initial firmware works...
Parts:
- removed D?: 1N4001, Diode_THT:D_DO-41_SOD81_P10.16mm_Horizontal, symbol Diode:1N4001
- removed D?: LED, symbol Device:LED
- removed D?: BAND_SPLIT, symbol Device:LED
- removed K?: G6E, Relay_THT:Relay_SPDT_Omron_G6E, symbol Relay:G6E
- removed Q?: BT169B, Package_TO_SOT_THT:TO-92_Inline, symbol Triac_Thyristor:BT169B
- removed R? (x2): R_Small_US, symbol Device:R_Small_US
- removed R?: 1K, symbol Device:R_Small_US
- removed RV?: R_Potentiometer_US, symbol Device:R_Potentiometer_US
- removed TP?: WDT Out, symbol Connector:TestPoint_Alt
- removed U?: LM555xM, Package_SO:SOIC-8_3.9x4.9mm_P1.27mm, symbol Timer:LM555xM
- gave numbers to parts that had none: 30
Other:
- note removed: "FRONTEND"
- note removed: "Fine Adjust"
- note removed: "HIGH"
- note removed: "High Band"
- note removed: "LOW"
- note removed: "LOW/HI BAND"
- note removed: "TX Watchdog"
- note removed: "To prevent runaway TX, require host CPU to toggle WD pin >100ms, before timeout. This should be rather lengthy, perhaps 5-10 minutes, as it will define the maximum allowed TX time in self-hosted modes. This should have a direct unmuxed GPIO pin"
- note removed: "WDT Triggered"
