File: control_logic.kicad_sch (KiCad schematic)
At the start: 28 parts, among them J20 USB_A_Stacked, J21 USB, J22 CTRL:PA_L, J23 CTRL:PA_H, J24 CTRL:FILT_L, J25 CTRL:FILT_H, J26 CTRL:ATU_L, J27 CTRL:ATU_H, U10 TUSB4041I, U11 STM32 Blackpill, Y1 24Mhz

Commit message: cleanup and trying to implement stubs for future features
Connections:
- net at U10.33 (USB_DP_DN1): now also JP2.1 (A); no longer JP2.2 (C)
- net at U10.34 (USB_DM_DN1): now also JP1.1 (A); no longer JP1.2 (C)
- net at R64.2: now also JP2.3 (B); no longer JP2.1 (A)
- net at JP4.3 (B): now also JP2.2 (C); no longer JP2.3 (B)
- net at JP3.3 (B): now also JP1.2 (C); no longer JP1.3 (B)
- net at R65.2: now also JP1.3 (B); no longer JP1.1 (A)
Other:
- moved on the sheet: JP1, JP2
Changed lines of the file:
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@@
     (stroke (width 0) (type default) (color 132 132 0 1))
   )
+  (wire (pts (xy 222.25 29.21) (xy 265.43 29.21))
+    (stroke (width 0) (type default))
+  )
   (wire (pts (xy 232.41 157.48) (xy 228.6 157.48))
     (stroke (width 0) (type default))
   )
   (polyline (pts (xy 171.45 111.76) (xy 171.45 111.76))
-    (stroke (width 0) (type default))
-  )
-  (wire (pts (xy 269.24 20.32) (xy 269.24 39.37))
     (stroke (width 0) (type default))
   )
@@
     (stroke (width 0) (type default))
   )
-  (wire (pts (xy 212.09 116.84) (xy 212.09 25.4))
+  (wire (pts (xy 212.09 116.84) (xy 212.09 24.13))
     (stroke (width 0) (type default))
   )
@@
     (stroke (width 0) (type default) (color 132 0 0 1))
   )
-  (wire (pts (xy 212.09 25.4) (xy 217.17 25.4))
+  (wire (pts (xy 212.09 24.13) (xy 218.44 24.13))
     (stroke (width 0) (type default))
   )
@@
     (stroke (width 0) (type default) (color 132 0 0 1))
   )
-  (wire (pts (xy 227.33 25.4) (xy 265.43 25.4))
-    (stroke (width 0) (type default))
-  )
   (wire (pts (xy 209.55 128.27) (xy 209.55 120.65))
     (stroke (width 0) (type default))
@@
     (stroke (width 0) (type default))
   )
+  (wire (pts (xy 229.87 26.67) (xy 229.87 22.86))
+    (stroke (width 0) (type default))
+  )
   (wire (pts (xy 193.04 165.1) (xy 218.44 165.1))
     (stroke (width 0) (type default))
@@
     (stroke (width 0) (type default) (color 255 153 0 1))
   )
+  (wire (pts (xy 210.82 17.78) (xy 226.06 17.78))
+    (stroke (width 0) (type default))
+  )
   (wire (pts (xy 25.4 138.43) (xy 27.94 138.43))
     (stroke (width 0) (type default))
@@
     (stroke (width 0) (type default))
   )
-  (wire (pts (xy 236.22 20.32) (xy 269.24 20.32))
-    (stroke (width 0) (type default))
-  )
   (wire (pts (xy 191.77 163.83) (xy 219.71 163.83))
     (stroke (width 0) (type default))
@@
     (stroke (width 0) (type default) (color 255 153 0 1))
   )
-  (wire (pts (xy 222.25 13.97) (xy 222.25 21.59))
-    (stroke (width 0) (type default))
-  )
   (wire (pts (xy 236.22 96.52) (xy 236.22 91.44))
     (stroke (width 0) (type default) (color 255 255 0 1))
@@
     (stroke (width 0) (type default) (color 255 153 0 1))
   )
-  (wire (pts (xy 265.43 25.4) (xy 265.43 39.37))
+  (wire (pts (xy 265.43 29.21) (xy 265.43 39.37))
     (stroke (width 0) (type default))
   )
@@
     (stroke (width 0) (type default))
   )
+  (wire (pts (xy 229.87 26.67) (xy 269.24 26.67))
+    (stroke (width 0) (type default))
+  )
   (wire (pts (xy 265.43 44.45) (xy 265.43 50.8))
     (stroke (width 0) (type default))
@@
     (stroke (width 0) (type default) (color 255 153 0 1))
   )
+  (wire (pts (xy 222.25 13.97) (xy 222.25 19.05))
+    (stroke (width 0) (type default))
+  )
   (wire (pts (xy 186.69 41.91) (xy 186.69 59.69))
     (stroke (width 0) (type default))
@@
     (stroke (width 0) (type default))
   )
-  (wire (pts (xy 45.72 12.7) (xy 231.14 12.7))
-    (stroke (width 0) (type default))
-  )
-  (wire (pts (xy 210.82 20.32) (xy 226.06 20.32))
+  (wire (pts (xy 45.72 12.7) (xy 229.87 12.7))
     (stroke (width 0) (type default))
   )
@@
     (stroke (width 0) (type default) (color 255 153 0 1))
   )
+  (wire (pts (xy 269.24 26.67) (xy 269.24 39.37))
+    (stroke (width 0) (type default))
+  )
   (wire (pts (xy 251.46 76.2) (xy 256.54 76.2))
     (stroke (width 0) (type default))
@@
     (stroke (width 0) (type default) (color 132 132 0 1))
   )
-  (wire (pts (xy 231.14 12.7) (xy 231.14 16.51))
-    (stroke (width 0) (type default))
-  )
   (wire (pts (xy 208.28 130.81) (xy 210.82 130.81))
     (stroke (width 0) (type default) (color 132 0 0 1))
@@
     (stroke (width 0) (type default))
   )
-  (wire (pts (xy 210.82 20.32) (xy 210.82 111.76))
+  (wire (pts (xy 210.82 17.78) (xy 210.82 111.76))
     (stroke (width 0) (type default))
   )
@@
     )
   )
-  (symbol (lib_id "Jumper:SolderJumper_3_Open") (at 222.25 25.4 180) (unit 1)
-    (in_bom yes) (on_board yes) (dnp no)
-    (property "Reference" "JP2" (at 214.63 21.59 0)
-      (effects (font (size 1.27 1.27)))
-    )
-    (property "Value" "USB_DP" (at 215.9 24.13 0)
-      (effects (font (size 1.27 1.27)))
-    )
-    (property "Footprint" "" (at 222.25 25.4 0)
-      (effects (font (size 1.27 1.27)) hide)
-    )
-    (property "Datasheet" "~" (at 222.25 25.4 0)
+  (symbol (lib_id "Jumper:SolderJumper_3_Open") (at 222.25 24.13 270) (unit 1)
+    (in_bom yes) (on_board yes) (dnp no)
+    (property "Reference" "JP2" (at 218.44 31.75 0)
+      (effects (font (size 1.27 1.27)))
+    )
+    (property "Value" "USB_DP" (at 220.98 30.48 0)
+      (effects (font (size 1.27 1.27)))
+    )
+    (property "Footprint" "" (at 222.25 24.13 0)
+      (effects (font (size 1.27 1.27)) hide)
+    )
+    (property "Datasheet" "~" (at 222.25 24.13 0)
       (effects (font (size 1.27 1.27)) hide)
     )
@@
     )
   )
-  (symbol (lib_id "Jumper:SolderJumper_3_Open") (at 231.14 20.32 180) (unit 1)
-    (in_bom yes) (on_board yes) (dnp no)
-    (property "Reference" "JP1" (at 234.95 15.24 0)
-      (effects (font (size 1.27 1.27)))
-    )
-    (property "Value" "USB_DM" (at 237.2042 17.7156 0)
-      (effects (font (size 1.27 1.27)))
-    )
-    (property "Footprint" "" (at 231.14 20.32 0)
-      (effects (font (size 1.27 1.27)) hide)
-    )
-    (property "Datasheet" "~" (at 231.14 20.32 0)
-      (effects (font (size 1.27 1.27)) hide)
-    )
+  (symbol (lib_id "Jumper:SolderJumper_3_Open") (at 229.87 17.78 270) (unit 1)
+    (in_bom yes) (on_board yes) (dnp no)
+    (property "Reference" "JP1" (at 227.3944 4.7942 0)
+      (effects (font (size 1.27 1.27)))
+    )
+    (property "Value" "USB_DM" (at 229.87 2.54 0)
+      (effects (font (size 1.27 1.27)))
+    )
+    (property "Footprint" "" (at 229.87 17.78 0)
+      (effects (font (size 1.27 1.27)) hide)
+    )
+    (property "Datasheet" "~" (at 229.87 17.78 0)
+      (effects (font (size 1.27 1.27)) hide)
+    )
