File: pcb/radiopcb.kicad_pcb (KiCad board)
At the start: 2 copper layers, 165 parts, among them J21 USB, K1 EC2-5SNU, K10 EC2-5SNU, K11 EC2-5SNU, K12 EC2-5SNU, K13 EC2-5SNU, K14 G6E, K15 G6E, K16 G6E, K17 G6E, K18 G6E, K19 G6E, K2 EC2-5SNU, K20 G6E, K21 G6E, K22 G6E, K23 G6E, K24 G6E, K25 G6E, K26 G6E, K27 G6E, K28 G6E, K29 G6E, K3 EC2-5SNU, K30 G6E, K31 EC2-5SNU, K32 EC2-5SNU, K33 EC2-5SNU, K34 EC2-5SNU, K35 EC2-5SNU, K36 EC2-5SNU, K37 EC2-5SNU, K38 EC2-5SNU, K39 EC2-5SNU, K4 EC2-5SNU, K40 EC2-5SNU, K41 EC2-5SNU, K42 EC2-5SNU, K43 G6E, K44 EC2-5SNU, K45 EC2-5SNU, K5 EC2-5SNU, K6 EC2-5SNU, K7 EC2-5SNU, K8 EC2-5SNU, K9 EC2-5SNU, Q10 BT169B, Q9 2N3904, U10 TUSB4041I, U15 ULN2804A, U16 74HC596, U18 MCP23008-xSO, U19 LM555xM, U2 MCP23017_SO, U4 MCP23017_SO, U7 MCP23008-xSO, U9 CM119B, Y1 24Mhz

Commit message: cleanup
Parts:
- moved K45 97.0 mm to (92.4, 62.9)
- moved K1 96.7 mm to (79.4, 63.9)
- moved F1 38.9 mm to (162.0, 14.3)
