File: pcb/hf_atu.kicad_sch (KiCad schematic)
At the start: 119 parts, among them J10 To CTRL:ATU, J11 TO TX_FILT_OUT, J12 TO SWR_IN, J8 SWR_IN, J9 SWR_OUT, K14 G6E, K15 G6E, K16 G6E, K17 G6E, K18 G6E, K19 G6E, K20 G6E, K21 G6E, K22 G6E, K23 G6E, K24 G6E, K25 G6E, K26 G6E, K27 G6E, K28 G6E, K29 G6E, K30 G6E, T1 SWR, U4 MCP23017_SO, U5 ULN2803A, U6 ULN2803A, U7 MCP23008-xSO, U8 ULN2803A

Commit message: cleanup of layout (fixed pcb/ subdirs; stubs for timers
Parts:
- removed C40: 100, symbol Device:C_Small
- removed C41, C43, C45, C46: 0.01, symbol Device:C_Small
- removed C42: 3-23, symbol Device:C_Variable
- removed C44, C62: 0.1u, Capacitor_THT:C_Disc_D4.7mm_W2.5mm_P5.00mm, symbol Device:C_Small
- removed C47, C55, C63: 100u, symbol Device:C_Polarized_Small
- removed C48, C52: 82p, symbol Device:C_Small
- removed C49: 220p, symbol Device:C_Small
- removed C50: 100p, symbol Device:C_Small
- removed C51: 560p, symbol Device:C_Small
- removed C53: 150p, symbol Device:C_Small
- removed C54, C56, C58, C59, C60, C61: 10p, symbol Device:C_Small
- removed C57: 39p, symbol Device:C_Small
- removed D14, D15: 1N4148, Diode_THT:D_DO-35_SOD27_P7.62mm_Horizontal, symbol Diode:1N4148
- removed D16: AT-82pF, symbol Device:LED
- removed D17: AT-160pF, symbol Device:LED
- removed D18: AT-320pF, symbol Device:LED
- removed D19: AT-642pF, symbol Device:LED
- removed D20, D21, D22, D27, D28, D29: LED, symbol Device:LED
- removed D23: AT-5pF, symbol Device:LED
- removed D24: AT-10pF, symbol Device:LED
- removed D25: AT-20pF, symbol Device:LED
- removed D26: AT-39pF, symbol Device:LED
- removed D30: HiZ-Green, symbol Device:LED
- removed D31: Bypass-Red, symbol Device:LED
- removed D32: AT-1.25uH, symbol Device:LED
- removed D33: AT-2.5uH, symbol Device:LED
- removed D34: AT-5.0uH, symbol Device:LED
- removed D35: AT-10uH, symbol Device:LED
- removed D36: AT-0.22uH, symbol Device:LED
- removed D37: AT-0.39uH, symbol Device:LED
- removed D38: AT-0.59uH, symbol Device:LED
- removed D39: AT-0.11uH, symbol Device:LED
- removed J10: To CTRL:ATU, symbol Connector_Generic:Conn_2Rows-09Pins
- removed J11: TO TX_FILT_OUT, symbol Connector:Conn_Coaxial
- removed J12: TO SWR_IN, symbol Connector:Conn_Coaxial
- removed J8: SWR_IN, symbol Connector:Conn_Coaxial
- removed J9: SWR_OUT, symbol Connector:Conn_Coaxial
- removed K14, K15, K16, K17, K18, K19, K20, K21, K22, K23, K24, K25, K26, K27, K28, K29, K30: G6E, Relay_THT:Relay_SPDT_Omron_G6E, symbol Relay:G6E
- removed L31: 1.25u, symbol Device:L_Ferrite
- removed L32: 2.5u, symbol Device:L_Ferrite
- removed L33: 5.0u, symbol Device:L_Ferrite
- removed L34: 10u, symbol Device:L_Ferrite
- removed L35: 0.22u, symbol Device:L_Ferrite
- removed L36: 0.39u, symbol Device:L_Ferrite
- removed L37: 0.59u, symbol Device:L_Ferrite
- removed L38: 0.11u, symbol Device:L_Ferrite
- removed R14: 3.3k, symbol Device:R_Small_US
- removed R15, R17: 100, symbol Device:R_Small_US
- removed R16: 150, symbol Device:R_Small_US
- removed R18, R19, R20, R21, R22, R23, R24, R25, R26, R27, R28, R29, R30, R31, R34, R35, R36, R37, R38, R39, R40, R41: 10K, symbol Device:R_Small_US
- removed R32, R33: 10k, symbol Device:R_Small_US
- removed RL1: Bypass, Relay_THT:Relay_DPDT_Panasonic_JW2, symbol Relay:JW2
- removed RV1, RV2: 100k, symbol Device:R_Potentiometer_US
- removed T1: SWR, symbol Device:Transformer_1P_SS
- removed TP1: REV_SWR, symbol Connector:TestPoint
- removed TP2: FWD_SWR, symbol Connector:TestPoint
- removed U4: MCP23017_SO, Package_SO:SOIC-28W_7.5x17.9mm_P1.27mm, symbol Interface_Expansion:MCP23017_SO
- removed U5, U6, U8: ULN2803A, symbol Transistor_Array:ULN2803A
- removed U7: MCP23008-xSO, Package_SO:SOIC-18W_7.5x11.6mm_P1.27mm, symbol Interface_Expansion:MCP23008-xSO
Connections:
- no-connect marks 26 -> 0
Other:
- note removed: "1: REV_SWR 2: 3: FWD_SWR 4: +12V 5: i2c SDA 6: GND 7: i2c SCK 8: +5V 9:"
- note removed: "BYPASS"
- note removed: "HI-Z"
- note removed: "L/C values derived from published LDG AT-11 manual. RF path designed to minimize # of relays needed Board interconnections via SMA connections."
- note removed: "SWR BRIDGE"
- note removed: "i2c addr: 0x01"
- note removed: "i2c addr: 0x02"
- note removed: "status lights"
