File: pcb/RAT50/RAT50/RAT50.kicad_sch (KiCad schematic)
At the start: 119 parts, among them J10 To CTRL:ATU, J11 TO TX_FILT_OUT, J12 TO SWR_IN, J8 SWR_IN, J9 SWR_OUT, K14 G6E, K15 G6E, K16 G6E, K17 G6E, K18 G6E, K19 G6E, K20 G6E, K21 G6E, K22 G6E, K23 G6E, K24 G6E, K25 G6E, K26 G6E, K27 G6E, K28 G6E, K29 G6E, K30 G6E, T1 SWR, U4 MCP23017_SO, U5 ULN2803A, U6 ULN2803A, U7 MCP23008-xSO, U8 ULN2803A

Commit message: cleanup
Parts:
- removed C40: 100, symbol Device:C_Small
- removed C41, C43, C45, C46: 0.01, symbol Device:C_Small
- removed C42: 3-23, symbol Device:C_Variable
- removed C44, C62: 0.1u, Capacitor_THT:C_Disc_D4.7mm_W2.5mm_P5.00mm, symbol Device:C_Small
- removed C47, C55, C63: 100u, symbol Device:C_Polarized_Small
- removed C48, C52: 82p, symbol Device:C_Small
- removed C49: 220p, symbol Device:C_Small
- removed C50: 100p, symbol Device:C_Small
- removed C51: 560p, symbol Device:C_Small
- removed C53: 150p, symbol Device:C_Small
- removed C54, C56, C58, C59, C60, C61: 10p, symbol Device:C_Small
- removed C57: 39p, symbol Device:C_Small
- removed D14, D15: 1N4148, Diode_THT:D_DO-35_SOD27_P7.62mm_Horizontal, symbol Diode:1N4148
- removed D27, D28, D29: LED, symbol Device:LED
- removed D30: HiZ-Green, symbol Device:LED
- removed D31: Bypass-Red, symbol Device:LED
- removed D32: AT-1.25uH, symbol Device:LED
- removed D33: AT-2.5uH, symbol Device:LED
- removed D34: AT-5.0uH, symbol Device:LED
- removed D35: AT-10uH, symbol Device:LED
- removed D36: AT-0.22uH, symbol Device:LED
- removed D37: AT-0.39uH, symbol Device:LED
- removed D38: AT-0.59uH, symbol Device:LED
- removed D39: AT-0.11uH, symbol Device:LED
- removed J10: To CTRL:ATU, symbol Connector_Generic:Conn_2Rows-09Pins
- removed J11: TO TX_FILT_OUT, symbol Connector:Conn_Coaxial
- removed J12: TO SWR_IN, symbol Connector:Conn_Coaxial
- removed J8: SWR_IN, symbol Connector:Conn_Coaxial
- removed J9: SWR_OUT, symbol Connector:Conn_Coaxial
- removed K18, K19, K20, K21, K22, K23, K24, K25, K26, K27, K28, K29, K30: G6E, Relay_THT:Relay_SPDT_Omron_G6E, symbol Relay:G6E
- removed L31: 1.25u, symbol Device:L_Ferrite
- removed L32: 2.5u, symbol Device:L_Ferrite
- removed L33: 5.0u, symbol Device:L_Ferrite
- removed L34: 10u, symbol Device:L_Ferrite
- removed L35: 0.22u, symbol Device:L_Ferrite
- removed L36: 0.39u, symbol Device:L_Ferrite
- removed L37: 0.59u, symbol Device:L_Ferrite
- removed L38: 0.11u, symbol Device:L_Ferrite
- removed R29, R30, R31, R34, R35, R36, R37, R38, R39, R40, R41: 10K, symbol Device:R_Small_US
- removed R32, R33: 10k, symbol Device:R_Small_US
- removed U4: MCP23017_SO, Package_SO:SOIC-28W_7.5x17.9mm_P1.27mm, symbol Interface_Expansion:MCP23017_SO
- removed U6, U8: ULN2803A, symbol Transistor_Array:ULN2803A
- removed U7: MCP23008-xSO, Package_SO:SOIC-18W_7.5x11.6mm_P1.27mm, symbol Interface_Expansion:MCP23008-xSO
- added C1: 100, symbol Device:C_Small
- added C10: 220p, symbol Device:C_Small
- added C11: 100p, symbol Device:C_Small
- added C12: 560p, symbol Device:C_Small
- added C13, C9: 82p, symbol Device:C_Small
- added C14: 150p, symbol Device:C_Small
- added C15, C17, C19, C20, C21, C22: 10p, symbol Device:C_Small
- added C16, C24, C8: 100u, symbol Device:C_Polarized_Small
- added C18: 39p, symbol Device:C_Small
- added C2, C4, C6, C7: 0.01, symbol Device:C_Small
- added C23, C5: 0.1u, Capacitor_THT:C_Disc_D4.7mm_W2.5mm_P5.00mm, symbol Device:C_Small
- added C3: 3-23, symbol Device:C_Variable
- added D1, D2: 1N4148, Diode_THT:D_DO-35_SOD27_P7.62mm_Horizontal, symbol Diode:1N4148
- added D10: AT-5pF, symbol Device:LED
- added D11: AT-10pF, symbol Device:LED
- added D12: AT-20pF, symbol Device:LED
- added D13: AT-39pF, symbol Device:LED
- added D14, D15, D7, D8, D9: LED, symbol Device:LED
- added D3: AT-82pF, symbol Device:LED
- added D4: AT-160pF, symbol Device:LED
- added D5: AT-320pF, symbol Device:LED
- added D6: AT-642pF, symbol Device:LED
- added J1: SWR_IN, symbol Connector:Conn_Coaxial
- added J2: SWR_OUT, symbol Connector:Conn_Coaxial
- added J3: To CTRL:ATU, symbol Connector_Generic:Conn_2Rows-09Pins
- added J4: TO TX_FILT_OUT, symbol Connector:Conn_Coaxial
- added J5: TO SWR_IN, symbol Connector:Conn_Coaxial
- added K1, K10, K11, K12, K13, K2, K3, K4, K5, K6, K7, K8, K9: G6E, Relay_THT:Relay_SPDT_Omron_G6E, symbol Relay:G6E
- added L1: 1.25u, symbol Device:L_Ferrite
- added L2: 2.5u, symbol Device:L_Ferrite
- added L3: 5.0u, symbol Device:L_Ferrite
- added L4: 10u, symbol Device:L_Ferrite
- added L5: 0.39u, symbol Device:L_Ferrite
- added L6: 0.22u, symbol Device:L_Ferrite
- added L7: 0.59u, symbol Device:L_Ferrite
- added L8: 0.11u, symbol Device:L_Ferrite
- added R1: 3.3k, symbol Device:R_Small_US
- added R10, R11, R12, R13, R5, R6, R7, R8, R9: 10K, symbol Device:R_Small_US
- added R2, R4: 100, symbol Device:R_Small_US
- added R3: 150, symbol Device:R_Small_US
- added U1: MCP23017_SO, Package_SO:SOIC-28W_7.5x17.9mm_P1.27mm, symbol Interface_Expansion:MCP23017_SO
- added U2, U3: ULN2803A, symbol Transistor_Array:ULN2803A
- added U4: MCP23008-xSO, Package_SO:SOIC-18W_7.5x11.6mm_P1.27mm, symbol Interface_Expansion:MCP23008-xSO
- D16: value AT-82pF -> LED
- D17: value AT-160pF -> HiZ-Green
- D18: value AT-320pF -> Bypass-Red
- D19: value AT-642pF -> AT-1.25uH
- D20: value LED -> AT-2.5uH
- D21: value LED -> AT-5.0uH
- D22: value LED -> AT-10uH
- D23: value AT-5pF -> AT-0.22uH
- D24: value AT-10pF -> AT-0.39uH
- D25: value AT-20pF -> AT-0.59uH
- D26: value AT-39pF -> AT-0.11uH
- R14: value 3.3k -> 10K
- R15, R17: value 100 -> 10K
- R16: value 150 -> 10K
- R19, R20: value 10K -> 10k
Connections:
- net +12V: now also R20.1, C16.1, C24.1, C8.1, D10.2 (A), D11.2 (A), D12.2 (A), D13.2 (A), D14.2 (A), D15.2 (A), D3.2 (A), D4.2 (A), D5.2 (A), D6.2 (A), D7.2 (A), D8.2 (A), D9.2 (A), J3.4 (Pin_4), K1.1, K10.1, K11.1, K12.1, K13.1, K2.1, K3.1, K4.1, K5.1, K6.1, K7.1, K8.1, K9.1, U2.10 (COM), U3.10 (COM); no longer D18.2 (A)
- net +5V: now also C23.2, C5.2, J3.8 (Pin_8), U1.15 (A0), U1.9 (VDD), U4.18 (VDD), U4.3 (A2), U4.4 (A1)
- net Earth: now also C1.2, C10.2, C11.2, C12.2, C13.2, C14.2, C15.2, C16.2, C17.2, C18.2, C2.2, C20.2, C21.2, C22.2, C23.1, C24.2, C4.2, C5.1, C6.2, C7.2, C8.2, C9.2, J1.2 (Ext), J2.2 (Ext), J3.2 (Pin_2), J3.6 (Pin_6), J3.9 (Pin_9), J4.2 (Ext), J5.2 (Ext), R1.2, U1.10 (VSS), U1.16 (A1), U1.17 (A2), U2.9 (GND), U3.9 (GND), U4.5 (A0), U4.9 (VSS); no longer R14.2
- net at RL1.3: now also J5.1 (In)
- net at RV2.2, TP2.1: now also C6.1, J3.3 (Pin_3)
- net at RL1.5: now also K16.7, K13.7, K9.10, L4.2, L7.2
- net at RL1.6: now also J4.1 (In)
- net at R27.1: now also K16.6, U5.15 (O4); no longer U5.16 (O3)
- net at R17.1: now also U3.14 (O5)
- net at R16.2: now also D14.1 (K); no longer T1.3 (SA)
- net at RV1.2, TP1.1: now also C4.1, J3.1 (Pin_1)
- net at R22.1: now also U5.13 (O6), K11.6
- net at R28.1: now also K17.6, U5.18 (O1); no longer U5.15 (O4)
- net at R15.1: now also K8.6, U2.15 (O4)
- net at T1.5 (SB): now also D1.2 (A), R3.1; no longer R16.1
- net at RL1.4: now also K12.7, K9.12, L3.2
- net at RL1.8: now also D18.1 (K), U3.11 (O8)
- net at U5.1 (I1): now also U4.10 (GP0)
- net at U5.2 (I2): now also U4.11 (GP1)
- net at U5.3 (I3): now also U4.12 (GP2)
- net at U5.4 (I4): now also U4.13 (GP3)
- net at U5.5 (I5): now also U4.14 (GP4)
- net at U5.6 (I6): now also U4.15 (GP5)
- net at U5.7 (I7): now also U4.16 (GP6)
- net at U5.8 (I8): now also U4.17 (GP7)
- net at R24.1: now also U5.11 (O8), K13.6
- net at R23.1: now also U5.12 (O7), K12.6
- net at R25.1: now also K14.6, U5.17 (O2); no longer U5.18 (O1)
- net at R14.1: now also K7.6, U2.16 (O3); no longer T1.4 (SC)
- net at T1.1 (AA): now also C3.1, J2.1 (In)
- net at R26.1: now also K15.6, U5.16 (O3); no longer U5.17 (O2)
- net at T1.2 (AB): now also J1.1 (In)
- net at R17.2: now also D15.1 (K); no longer RV2.1
- net at K17.10: now also L8.1
- net at R15.2: now also D13.1 (K); no longer RV1.1
- net at K16.10: now also K15.7, L5.2, L7.1
- net at K15.10: now also K14.7, L5.1, L6.2
- net at R20.2: now also D18.2 (A); no longer D18.1 (K)
- net at K14.10: now also K17.7, K10.10, L1.2, L6.1, L8.2
- new net: D12.1 (K), R14.2
- new net: C2.1, D1.1 (K), R2.1
- new net: K2.6, R6.1, U2.13 (O6)
- new net: D4.1 (K), R6.2
- new net: K11.7, K12.10, L2.1, L3.1
- new net: K10.7, K11.10, L1.1, L2.2
- new net: D10.1 (K), R12.2
- new net: D3.1 (K), R5.2
- new net: K9.6, R19.1, U3.12 (O7)
- new net: K1.7, K2.7, K3.7, K4.7, K5.7, K6.7, K7.7, K8.7, K9.7
- new net: C1.1, C3.2, R1.1, T1.4 (SC)
- new net: U1.1 (GPB0), U3.1 (I1)
- new net: J3.7 (Pin_7), U1.12 (SCK), U4.1 (SCL)
- new net: J3.5 (Pin_5), U1.13 (SDA), U4.2 (SDA)
- new net: U1.2 (GPB1), U3.2 (I2)
- new net: U1.21 (GPA0), U2.1 (I1)
- new net: U1.22 (GPA1), U2.2 (I2)
- new net: U1.23 (GPA2), U2.3 (I3)
- new net: U1.24 (GPA3), U2.4 (I4)
- new net: U1.25 (GPA4), U2.5 (I5)
- new net: U1.26 (GPA5), U2.6 (I6)
- new net: U1.27 (GPA6), U2.7 (I7)
- new net: U1.28 (GPA7), U2.8 (I8)
- new net: U1.3 (GPB2), U3.3 (I3)
- new net: U1.4 (GPB3), U3.4 (I4)
- new net: U1.5 (GPB4), U3.5 (I5)
- new net: U1.6 (GPB5), U3.6 (I6)
- new net: U1.7 (GPB6), U3.7 (I7)
- new net: U1.8 (GPB7), U3.8 (I8)
- new net: R9.1, U3.18 (O1)
- new net: D7.1 (K), R9.2
- new net: K10.6, R21.1, U5.14 (O5)
- new net: C10.1, C11.1, K3.12
- new net: D6.1 (K), R8.2
- new net: C17.1, K6.12
- new net: K3.6, R7.1, U2.12 (O7)
- new net: K6.6, R13.1, U2.17 (O2)
- new net: R16.1, U3.15 (O4)
- new net: C7.1, D2.1 (K), R4.1
- new net: D2.2 (A), R3.2, T1.3 (SA)
- new net: K4.6, R8.1, U2.11 (O8)
- new net: C20.1, C21.1, K7.12
- new net: K5.6, R12.1, U2.18 (O1)
- new net: C18.1, K8.12
- new net: C14.1, C15.1, K2.12
- new net: D5.1 (K), R7.2
- new net: R4.2, RV2.1
- new net: R18.1, U3.13 (O6)
- new net: R11.1, U3.16 (O3)
- new net: R10.1, U3.17 (O2)
- new net: D9.1 (K), R11.2
- new net: C12.1, C13.1, K4.12
- new net: C19.1, K5.12
- new net: D11.1 (K), R13.2
- new net: D8.1 (K), R10.2
- new net: C19.2, C22.1
- new net: K1.6, R5.1, U2.14 (O5)
- new net: R2.2, RV1.1
- new net: K13.10, L4.1
- new net: C9.1, K1.12
- no-connect marks 26 -> 21
Other:
- note added: "1: REV_SWR 2: GND 3: FWD_SWR 4: +12V 5: i2c SDA 6: GND 7: i2c SCK 8: +5V 9: GND"
- note added: "L/C values derived from published LDG AT-11 manual. RF path designed to minimize # of relays needed Board interconnections via SMA connections. We are intended for 50W at 100% duty cycle (digi, etc) or 100W on SSB."
- note removed: "1: REV_SWR 2: 3: FWD_SWR 4: +12V 5: i2c SDA 6: GND 7: i2c SCK 8: +5V 9:"
- note removed: "L/C values derived from published LDG AT-11 manual. RF path designed to minimize # of relays needed Board interconnections via SMA connections."
- title: HF Antenna Matching Unit -> (none)
